File: Ellow.kicad_pcb (KiCad board)
At the start: 2 copper layers, 20.5 x 36.8 mm, 26 parts, among them J1 USB_C_Receptacle_USB2.0, J2 M_2_AKey_KB, J3 Conn_01x02_Female, J4 Conn_01x04_Female, J5 Conn_01x04_Female, Q1 A03407, Q2 A03407, U1 AP2112K-3.3, U2 E73-2G4M08S1C, U3 LN2054Y42AMR, Y1 32.768kHz

Commit message: routing done, R0
Parts:
- removed J4: Conn_01x04_Female, ellow:PinHeader_1x04_P2.54mm_Vertical_small
- added H2: MountingHole, ellow:MountingHole_M.2_3mm, F.Cu at (225.3, 103.1)
- C1, R1, R2, R3, R6, R8: moved to F.Cu
- moved C2 10.3 mm to (243.6, 106.4), turned to 0 degrees
- moved U3 10.1 mm to (240.1, 109.9), turned to 180 degrees
- moved R7 8.72 mm to (230.2, 104.6), turned to 270 degrees
- moved R3 7.76 mm to (236.3, 103.7)
- moved R1 7.52 mm to (240.4, 103.7)
- moved R5 6.80 mm to (243.8, 109.5), turned to 180 degrees
- moved Q1 6.41 mm to (240.4, 106.2)
- moved R2 6.21 mm to (236.3, 105.1)
- moved R4 5.99 mm to (243.8, 108.0), turned to 0 degrees
- moved D1 5.60 mm to (236.9, 107.0), turned to 180 degrees
- moved R9 5.00 mm to (228.5, 94.6), turned to 90 degrees
- moved C1 4.96 mm to (233.8, 107.3)
- moved U1 4.62 mm to (235.9, 109.8), turned to 180 degrees
- moved R6 4.32 mm to (228.5, 99.3), turned to 270 degrees
- moved H1 4.17 mm to (245.8, 103.1)
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Connections:
- net Net-(U2-Pad15) renamed P0.05
- net Net-(U2-Pad17) renamed P1.09
- D2 pad 2: Net-(D2-Pad2) -> VBUS
- D3 pad 2: P0.07 -> P0.02
- J2 pad 1: GND -> Net-(J2-Pad1)
- J2 pad 23: Net-(J2-Pad23) -> P0.26
- J2 pad 27: Net-(J2-Pad27) -> P0.06
- J2 pad 31: Net-(J2-Pad31) -> P0.08
- J2 pad 35: Net-(J2-Pad35) -> P0.04
- J2 pad 38: Net-(J2-Pad38) -> P0.02
- J2 pad 39: Net-(J2-Pad39) -> P0.12
- J2 pad 43: Net-(J2-Pad43) -> P0.07
- J2 pad 46: Net-(J2-Pad46) -> P0.28
- J2 pad 5: VBAT -> Net-(J2-Pad5)
- J2 pad 50: Net-(J2-Pad50) -> P0.03
- J2 pad 6: Net-(J2-Pad6) -> GND
- J2 pad 62: Net-(J2-Pad62) -> P1.10
- J2 pad 66: Net-(J2-Pad66) -> P1.11
- R8 pad 1: Net-(R8-Pad1) -> PROG
- U2 pad 18: Net-(U2-Pad18) -> P0.04
- U2 pad 2: Net-(U2-Pad2) -> P1.10
- U3 pad 4: Net-(D2-Pad2) -> VBUS
- U3 pad 5: Net-(R8-Pad1) -> PROG
Routing:
- net P0.02: track 0.00 -> 47.8 mm, vias 0 -> 3
- net VBAT: track 46.4 -> 13.6 mm, vias 2 -> 0
- net PROG: track 0.00 -> 27.0 mm
- net Net-(R6-Pad2): track 7.33 -> 32.3 mm, vias 1 -> 0
- net P0.07: track 33.8 -> 10.4 mm, vias 1 -> 0
- net GND: track 19.2 -> 41.0 mm, vias 5 -> 7
- net P0.28: track 0.00 -> 19.6 mm
- net P1.10: track 0.00 -> 19.2 mm
- net P0.03: track 0.00 -> 19.1 mm
- net P1.11: track 0.00 -> 17.7 mm
- net P0.26: track 0.00 -> 16.7 mm
- net P0.06: track 0.00 -> 15.5 mm
- net P0.08: track 0.00 -> 14.3 mm
- net P0.04: track 0.00 -> 13.1 mm
- net P0.12: track 0.00 -> 11.9 mm
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Other:
- outline, holes or cut-outs redrawn

Commit message: EOD
Parts:
- moved R2 0.10 mm to (236.3, 105.2)
Connections:
- J2 pad 17: GND -> Net-(J2-Pad17)
Routing:
- net GND: track 41.0 -> 54.8 mm, vias 7 -> 11
- net EXT_VCC: track 10.9 -> 14.3 mm
